Commit message: Update URDF model colors, battery readout, and bump version to 2.1.7
Apply official TT Robotix RoboHero Iron Man red, gold, black,
and arc reactor cyan materials to the URDF model, replace
duplicate web public URDF with a symbolic link, display raw
integer battery telemetry, and bump project version to 2.1.7.

Co-authored-by: Gemini <gemini@google.com>
Signed-off-by: Charles Chiou <samurai@selfso.com>

File: urdf/robohero.urdf (robot description, URDF)
Before this commit: robot robohero, 18 links, 17 joints
Links:
- link base_link: geometry collision box size=0.055 0.076 0.080; visual box size=0.003 0.020 0.020
- link head_link: geometry collision box size=0.038 0.040 0.036; visual box size=0.002 0.016 0.016

Commit message: Fix URDF and kinematics joint mappings and bump version to 2.1.9
- Correct elbow joint axes in URDF to roll axis [1, 0, 0].
- Fix signs for right ankle roll, left hip roll, and elbows
  in RobotModel.js based on physical servo diagnostics.
- Bump project version to 2.1.9 across CMakeLists.txt and
  web package manifests.

Co-authored-by: Gemini <gemini@google.com>
Signed-off-by: Charles Chiou <samurai@selfso.com>

File: urdf/robohero.urdf (robot description, URDF)
Before this commit: robot robohero, 18 links, 17 joints
Joints:
- joint left_elbow_joint: axis 0 1 0 -> 1 0 0
- joint right_elbow_joint: axis 0 1 0 -> 1 0 0

Commit message: Calibrate 17 joints, update URDF limits and bump version to v2.1.10
- Empirically measure and calibrate angular limits for all 17 joints
- Update radPerPwm scaling constants in RobotModel.js
  (arms 135, legs 180)
- Encode measured lower and upper joint limits in urdf/robohero.urdf
- Document measurement methodology, results, and trim tables in doc/
- Bump project version to 2.1.10

Co-authored-by: Gemini <gemini@google.com>
Signed-off-by: Charles Chiou <samurai@selfso.com>

File: urdf/robohero.urdf (robot description, URDF)
Before this commit: robot robohero, 18 links, 17 joints
Joints:
- joint head_yaw_joint: limit lower=-1.5708 upper=1.5708 effort=0.8 velocity=3.14 -> lower=-1.3963 upper=1.3963 effort=0.8 velocity=3.14
- joint left_ankle_pitch_joint: limit lower=-1.5708 upper=1.5708 effort=1.5 velocity=3.14 -> lower=-0.7854 upper=1.5708 effort=1.5 velocity=3.14
- joint left_ankle_roll_joint: limit lower=-0.8727 upper=0.8727 effort=1.5 velocity=3.14 -> lower=-0.4363 upper=1.3090 effort=1.5 velocity=3.14
- joint left_elbow_joint: limit lower=-2.6180 upper=0.5236 effort=1.2 velocity=3.14 -> lower=-1.3090 upper=1.4835 effort=1.2 velocity=3.14
- joint left_hip_pitch_joint: limit lower=-1.5708 upper=1.5708 effort=1.5 velocity=3.14 -> lower=-0.6981 upper=1.5708 effort=1.5 velocity=3.14
- joint left_hip_roll_joint: limit lower=-0.6981 upper=0.8727 effort=1.5 velocity=3.14 -> lower=-0.3491 upper=1.6057 effort=1.5 velocity=3.14
- joint left_knee_pitch_joint: limit lower=-0.3491 upper=2.6180 effort=1.5 velocity=3.14 -> lower=-0.6981 upper=1.5708 effort=1.5 velocity=3.14
- joint left_shoulder_pitch_joint: limit lower=-3.1416 upper=3.1416 effort=1.2 velocity=3.14 -> lower=-3.1416 upper=1.5708 effort=1.2 velocity=3.14
- joint left_shoulder_roll_joint: limit lower=-0.3491 upper=2.6180 effort=1.2 velocity=3.14 -> lower=-0.0873 upper=2.9671 effort=1.2 velocity=3.14
- joint right_ankle_pitch_joint: limit lower=-1.5708 upper=1.5708 effort=1.5 velocity=3.14 -> lower=-0.8727 upper=1.5708 effort=1.5 velocity=3.14
- joint right_ankle_roll_joint: limit lower=-0.8727 upper=0.8727 effort=1.5 velocity=3.14 -> lower=-0.4363 upper=1.2217 effort=1.5 velocity=3.14
- joint right_elbow_joint: limit lower=-0.5236 upper=2.6180 effort=1.2 velocity=3.14 -> lower=-1.4835 upper=0.9599 effort=1.2 velocity=3.14
- joint right_hip_pitch_joint: limit lower=-1.5708 upper=1.5708 effort=1.5 velocity=3.14 -> lower=-0.6981 upper=1.5708 effort=1.5 velocity=3.14
- joint right_hip_roll_joint: limit lower=-0.8727 upper=0.6981 effort=1.5 velocity=3.14 -> lower=-1.7453 upper=0.3491 effort=1.5 velocity=3.14
- joint right_knee_pitch_joint: limit lower=-0.3491 upper=2.6180 effort=1.5 velocity=3.14 -> lower=-0.6981 upper=1.5708 effort=1.5 velocity=3.14
- joint right_shoulder_pitch_joint: limit lower=-3.1416 upper=3.1416 effort=1.2 velocity=3.14 -> lower=-1.5708 upper=2.0071 effort=1.2 velocity=3.14
- joint right_shoulder_roll_joint: limit lower=-2.6180 upper=0.3491 effort=1.2 velocity=3.14 -> lower=-2.9671 upper=0.0873 effort=1.2 velocity=3.14
