Commit message: Calibrated head for robot model
Signed-off-by: Charles Chiou <samurai@selfso.com>

File: urdf/robohero.urdf (robot description, URDF)
Before this commit: robot robohero, 18 links, 17 joints
Joints:
- joint head_yaw_joint: limit lower=-1.3963 upper=1.3963 effort=0.8 velocity=3.14 -> lower=-0.9756 upper=0.9233 effort=1.2 velocity=3.14

Commit message: Calibrated left/right shoulder pictch for model
Signed-off-by: Charles Chiou <samurai@selfso.com>

File: urdf/robohero.urdf (robot description, URDF)
Before this commit: robot robohero, 18 links, 17 joints
Joints:
- joint left_shoulder_pitch_joint: limit lower=-3.1416 upper=1.5708 effort=1.2 velocity=3.14 -> lower=-1.8117 upper=1.3055 effort=1.2 velocity=3.14
- joint right_shoulder_pitch_joint: limit lower=-1.5708 upper=2.0071 effort=1.2 velocity=3.14 -> lower=-2.4906 upper=2.0054 effort=1.2 velocity=3.14

Commit message: Calibrated left/right shoulder roll for model
Signed-off-by: Charles Chiou <samurai@selfso.com>

File: urdf/robohero.urdf (robot description, URDF)
Before this commit: robot robohero, 18 links, 17 joints
Joints:
- joint left_shoulder_roll_joint: limit lower=-0.0873 upper=2.9671 effort=1.2 velocity=3.14 -> lower=0.0000 upper=4.7298 effort=1.2 velocity=3.14
- joint right_shoulder_roll_joint: limit lower=-2.9671 upper=0.0873 effort=1.2 velocity=3.14 -> lower=-4.3284 upper=0.0000 effort=1.2 velocity=3.14
