Commit message: motion, model: fix left ankle roll limits and ghost telemetry
- Invert sign and expand limits for left ankle roll (Channel 0)
  in calibration.json and robohero.urdf to allow the full physical
  servo travel range (PWM 80-180, [-25 deg, 80 deg]).
- Maintain persistent telemetry arrays in Motion Studio MainWindow
  and only update channels with valid masks, preventing unmasked
  channels from resetting to 0 and distorting the ghost robot pose.
- Register std::array types as Qt meta-types and use QueuedConnection
  for cross-thread telemetry signal delivery.

Co-authored-by: Gemini <gemini@google.com>
Signed-off-by: Charles Chiou <samurai@selfso.com>

File: model/robohero.urdf (robot description, URDF)
Before this commit: robot robohero, 18 links, 17 joints
Joints:
- joint left_ankle_roll_joint: limit lower=-0.4363 upper=1.3090 effort=1.5 velocity=3.14 -> lower=-0.4363 upper=1.3963 effort=1.5 velocity=3.14

Commit message: motion, model, doc: fix ankle roll sign/limits and add duration spin
- Fix left ankle roll (Channel 0) sign to +1.0 and degree limits to
  [-80.0 deg, +25.0 deg] in model/calibration.json and robohero.urdf,
  correcting inverted physical rotation and restoring full travel.
- Add duration spin box (0.1s to 60.0s) in motion studio timeline to
  support motion sequences longer than default duration.
- Document raw PWM vs degree-bounded kinematic control paradigms across
  subprojects and bilateral roll symmetry conventions in doc/Model.md.
- Update empirical joint calibration records and guides across doc/.

Co-authored-by: Gemini <gemini@google.com>
Signed-off-by: Charles Chiou <samurai@selfso.com>

File: model/robohero.urdf (robot description, URDF)
Before this commit: robot robohero, 18 links, 17 joints
Joints:
- joint left_ankle_roll_joint: limit lower=-0.4363 upper=1.3963 effort=1.5 velocity=3.14 -> lower=-1.3963 upper=0.4363 effort=1.5 velocity=3.14
